File: KiCad/fertilizer-pump.kicad_sch (KiCad schematic)
At the start: 15 parts, among them U1 ESP32-S3-WROOM-1

Commit message: add valve driver, many changes
Parts:
- removed R3, R4: 10k, Resistor_SMD:R_0805_2012Metric_Pad1.20x1.40mm_HandSolder, symbol Device:R_Small
- added C29, C30: 100n, Capacitor_SMD:C_0805_2012Metric_Pad1.18x1.45mm_HandSolder, symbol Device:C_Small
- added R20, R21: 10K, Resistor_SMD:R_0805_2012Metric_Pad1.20x1.40mm_HandSolder, symbol Device:R_Small
- added SW1: BOOT, Library:SHOU HAN TS342A2P-WZ, symbol Switch:SW_Push
- added SW2: EN, Library:SHOU HAN TS342A2P-WZ, symbol Switch:SW_Push
- R1, R18, R19, R2: footprint (none) -> Resistor_SMD:R_0805_2012Metric_Pad1.20x1.40mm_HandSolder; LCSC (none) -> C2930231
Connections:
- net +3.3V: now also R20.2, R21.2
- net ESP_BOOT: now also C29.2, SW1.2
- net ESP_EN: now also C30.2, SW2.2
- net GND: now also C29.1, C30.1, SW1.1, SW2.1
- net I^{2}C.SCL: now also R20.1
- net I^{2}C.SDA: now also R21.1
- net SERVO4.PWM: now reaches U1.24 (GPIO47/SPICLK_P/SUBSPICLK_P_DIFF)
- net SERVO1.PWM: now reaches U1.31 (GPIO38/FSPIWP/SUBSPIWP)
- net SERVO2.PWM: now reaches U1.32 (MTCK/GPIO39/CLK_OUT3/SUBSPICS1)
- net SERVO3.PWM: now reaches U1.33 (MTDO/GPIO40/CLK_OUT2)
Other:
- note added: "servo output should be selectable via Solder bridge if there is a servo or a valve. Valve needs NMOS."
- moved on the sheet: C19, C20, C21, C22, R1, R14, R15, R16, R18, R19, R2, U1
