File: KiCad/fertilizer-pump.kicad_pcb (KiCad board)
At the start: 2 copper layers, 150 x 100 mm, 1 part

Commit message: .
Parts:
- added A2: BTT TMC2209, fertilizer-pump:BTT TMC2209, F.Cu at (129.6, 69.8)
- added C5: 1u, Capacitor_SMD:C_0805_2012Metric_Pad1.18x1.45mm_HandSolder, F.Cu at (210.3, 105.9)
- added C6: 1n, Capacitor_SMD:C_0805_2012Metric_Pad1.18x1.45mm_HandSolder, F.Cu at (210.3, 108.9)
- added D1: ESD762, Package_TO_SOT_SMD:SOT-23_Handsoldering, F.Cu at (187.7, 112.7)
- added D2: ESD762, Package_TO_SOT_SMD:SOT-23_Handsoldering, F.Cu at (187.7, 117.5)
- added D3: D_Zener, Diode_SMD:D_SOD-123F, F.Cu at (187.2, 121.4)
- added J1: Conn_01x04, Connector_JST:JST_XH_B4B-XH-A_1x04_P2.50mm_Vertical, F.Cu at (196.9, 107.7)
- added J2: Conn_01x04, Connector_JST:JST_XH_B4B-XH-A_1x04_P2.50mm_Vertical, F.Cu at (196.9, 115.5)
- added J6: USB_C_Receptacle_USB2.0_16P, Connector_USB:USB_C_Receptacle_GCT_USB4105-xx-A_16P_TopMnt_Horizontal, F.Cu at (178.6, 115.5)
- added R8: 10k, Resistor_SMD:R_0805_2012Metric_Pad1.20x1.40mm_HandSolder, F.Cu at (210.3, 111.9)
- added R9: 10k, Resistor_SMD:R_0805_2012Metric_Pad1.20x1.40mm_HandSolder, F.Cu at (210.3, 114.8)
- added U1: HUSB238_xxxDD, Package_DFN_QFN:WDFN-10-1EP_3x3mm_P0.5mm_EP1.8x2.5mm_ThermalVias, F.Cu at (210.9, 118.6)
- added U2: ESP32-S3-WROOM-1, PCM_Espressif:ESP32-S3-WROOM-1, F.Cu at (183.1, 99.1)
- A1: footprint Module:Pololu_Breakout-16_15.2x20.3mm -> fertilizer-pump:BTT TMC2209
- moved A1 18.9 mm to (112.8, 69.8)
Connections:
- A1 pad 1: unconnected-(A1-ENABLE-Pad1) -> DRIV.ENABLE
- A1 pad 10: (no net) -> +3.3V
- A1 pad 11: unconnected-(A1-B2-Pad11) -> DRIV1.B2
- A1 pad 12: unconnected-(A1-B1-Pad12) -> DRIV1.B1
- A1 pad 13: unconnected-(A1-A1-Pad13) -> DRIV1.A1
- A1 pad 14: unconnected-(A1-A2-Pad14) -> DRIV1.A2
- A1 pad 16: unconnected-(A1-VM-Pad16) -> +12V
- A1 pad 2: unconnected-(A1-MS1-Pad2) -> GND
- A1 pad 3: unconnected-(A1-MS2-Pad3) -> GND
- A1 pad 4: unconnected-(A1-PDN1-Pad4) -> DRIV.UART
- A1 pad 6: unconnected-(A1-CLK-Pad6) -> GND
- A1 pad 7: unconnected-(A1-STEP-Pad7) -> DRIV1.STEP
- A1 pad 8: unconnected-(A1-DIR-Pad8) -> DRIV1.DIR

Commit message: add valve driver, many changes
Parts:
- removed R9: 10k, Resistor_SMD:R_0805_2012Metric_Pad1.20x1.40mm_HandSolder
- removed the U1 at (210.9, 118.6)
- added A3: BTT TMC2209, fertilizer-pump:BTT TMC2209, F.Cu at (140.7, 79.1)
- added A4: BTT TMC2209, fertilizer-pump:BTT TMC2209, F.Cu at (140.7, 56.1)
- added C1: 220µF, Capacitor_SMD:CP_Elec_6.3x7.7, F.Cu at (199.0, 93.0)
- added C10: 22u, Capacitor_SMD:C_0805_2012Metric_Pad1.18x1.45mm_HandSolder, F.Cu at (172.6, 114.9)
- added C11: 220uF, Capacitor_THT:CP_Radial_D8.0mm_P3.50mm, F.Cu at (178.2, 103.2)
- added C12: 100n, Capacitor_SMD:C_0805_2012Metric_Pad1.18x1.45mm_HandSolder, F.Cu at (194.8, 116.0)
- added C13: 100n, Capacitor_SMD:C_0805_2012Metric_Pad1.18x1.45mm_HandSolder, F.Cu at (194.8, 119.0)
- added C14: 10u, Capacitor_SMD:C_0805_2012Metric_Pad1.18x1.45mm_HandSolder, F.Cu at (194.8, 122.0)
- added C15: 75p, Capacitor_SMD:C_0805_2012Metric_Pad1.18x1.45mm_HandSolder, F.Cu at (194.8, 125.1)
- added C16: 22u, Capacitor_SMD:C_0805_2012Metric_Pad1.18x1.45mm_HandSolder, F.Cu at (194.8, 128.1)
- added C17: 22u, Capacitor_SMD:C_0805_2012Metric_Pad1.18x1.45mm_HandSolder, F.Cu at (194.8, 131.1)
- added C18: 220uF, Capacitor_THT:CP_Radial_D8.0mm_P3.50mm, F.Cu at (200.4, 119.3)
- added C19: 1u, Capacitor_SMD:C_0805_2012Metric_Pad1.18x1.45mm_HandSolder, F.Cu at (86.4, 84.6)
- added C2: 100n, Capacitor_SMD:C_0805_2012Metric_Pad1.18x1.45mm_HandSolder, F.Cu at (201.5, 101.9)
- added C20: 22u, Capacitor_SMD:C_0805_2012Metric_Pad1.18x1.45mm_HandSolder, F.Cu at (86.4, 87.6)
- added C21: 10u, Capacitor_SMD:C_0805_2012Metric_Pad1.18x1.45mm_HandSolder, F.Cu at (86.4, 90.6)
- added C22: 100n, Capacitor_SMD:C_0805_2012Metric_Pad1.18x1.45mm_HandSolder, F.Cu at (86.4, 93.6)
- added C23: 220µF, Capacitor_SMD:CP_Elec_6.3x7.7, F.Cu at (198.5, 66.0)
- added C24: 100n, Capacitor_SMD:C_0805_2012Metric_Pad1.18x1.45mm_HandSolder, F.Cu at (201.0, 74.9)
- added C25: 220µF, Capacitor_SMD:CP_Elec_6.3x7.7, F.Cu at (160.5, 88.0)
- added C26: 100n, Capacitor_SMD:C_0805_2012Metric_Pad1.18x1.45mm_HandSolder, F.Cu at (158.0, 79.1)
- added C27: 220µF, Capacitor_SMD:CP_Elec_6.3x7.7, F.Cu at (160.5, 65.0)
- added C28: 100n, Capacitor_SMD:C_0805_2012Metric_Pad1.18x1.45mm_HandSolder, F.Cu at (158.0, 56.1)
- added C29: 100n, Capacitor_SMD:C_0805_2012Metric_Pad1.18x1.45mm_HandSolder, F.Cu at (56.3, 52.4)
- added C3: 1u, Capacitor_SMD:C_0805_2012Metric_Pad1.18x1.45mm_HandSolder, F.Cu at (172.6, 130.7)
- added C30: 100n, Capacitor_SMD:C_0805_2012Metric_Pad1.18x1.45mm_HandSolder, F.Cu at (56.3, 55.4)
- added C4: 1n, Capacitor_SMD:C_0805_2012Metric_Pad1.18x1.45mm_HandSolder, F.Cu at (184.0, 148.5)
- added C7: 10u, Capacitor_SMD:C_0805_2012Metric_Pad1.18x1.45mm_HandSolder, F.Cu at (172.6, 105.9)
- added C8: 47p, Capacitor_SMD:C_0805_2012Metric_Pad1.18x1.45mm_HandSolder, F.Cu at (172.6, 108.9)
- added C9: 22u, Capacitor_SMD:C_0805_2012Metric_Pad1.18x1.45mm_HandSolder, F.Cu at (172.6, 111.9)
- added D4: SS14, Diode_SMD:D_SMA_Handsoldering, F.Cu at (154.0, 148.5)
- added D5: SS14, Diode_SMD:D_SMA_Handsoldering, F.Cu at (144.5, 148.5)
- added D6: SS14, Diode_SMD:D_SMA_Handsoldering, F.Cu at (163.5, 148.5)
- added D7: SS14, Diode_SMD:D_SMA_Handsoldering, F.Cu at (135.0, 148.5)
- added J11: Conn_01x02, Connector_JST:JST_XH_B2B-XH-A_1x02_P2.50mm_Vertical, F.Cu at (152.2, 141.0)
- added J12: Conn_01x02, Connector_JST:JST_XH_B2B-XH-A_1x02_P2.50mm_Vertical, F.Cu at (143.2, 141.0)
- added J13: Conn_01x02, Connector_JST:JST_XH_B2B-XH-A_1x02_P2.50mm_Vertical, F.Cu at (161.2, 141.0)
- added J14: Conn_01x02, Connector_JST:JST_XH_B2B-XH-A_1x02_P2.50mm_Vertical, F.Cu at (133.8, 141.0)
- added J15: Barrel_Jack_Switch, Connector_BarrelJack:BarrelJack_GCT_DCJ200-10-A_Horizontal, F.Cu at (196.8, 138.2)
- added J3: Stepper3, Connector_JST:JST_XH_B4B-XH-A_1x04_P2.50mm_Vertical, F.Cu at (134.0, 91.8)
- added J4: Stepper4, Connector_JST:JST_XH_B4B-XH-A_1x04_P2.50mm_Vertical, F.Cu at (134.0, 68.8)
- added J5: Servo1, Connector_JST:JST_XH_B3B-XH-A_1x03_P2.50mm_Vertical, F.Cu at (132.5, 124.5)
- added J7: Servo2, Connector_JST:JST_XH_B3B-XH-A_1x03_P2.50mm_Vertical, F.Cu at (143.5, 124.5)
- added J8: Servo3, Connector_JST:JST_XH_B3B-XH-A_1x03_P2.50mm_Vertical, F.Cu at (154.5, 124.5)
- added J9: Servo4, Connector_JST:JST_XH_B3B-XH-A_1x03_P2.50mm_Vertical, F.Cu at (165.5, 124.5)
- added JP1: SolderJumper_2_Open, Jumper:SolderJumper-2_P1.3mm_Open_RoundedPad1.0x1.5mm, F.Cu at (171.6, 134.7)
- added JP2: SolderJumper_2_Open, Jumper:SolderJumper-2_P1.3mm_Open_RoundedPad1.0x1.5mm, F.Cu at (171.6, 137.7)
- added JP3: Connect shield to GND, Jumper:SolderJumper-2_P1.3mm_Open_RoundedPad1.0x1.5mm, F.Cu at (90.7, 119.4)
- added JP8: VMotor source select, Jumper:SolderJumper-3_P1.3mm_Open_RoundedPad1.0x1.5mm, F.Cu at (177.8, 79.5)
- added JP9: VRegulator source select, Jumper:SolderJumper-3_P1.3mm_Open_RoundedPad1.0x1.5mm, F.Cu at (177.7, 85.0)
- added L1: 10u, Inductor_SMD:L_APV_APH0630, F.Cu at (180.0, 112.0)
- added L2: 10u, Inductor_SMD:L_APV_APH0630, F.Cu at (202.2, 128.2)
- added Q1: SI2307A, Package_TO_SOT_SMD:SOT-23, F.Cu at (176.1, 130.7)
- added Q2: AO3400A, Package_TO_SOT_SMD:SOT-23, F.Cu at (156.0, 135.0)
- added Q3: AO3400A, Package_TO_SOT_SMD:SOT-23, F.Cu at (146.5, 135.0)
- added Q4: AO3400A, Package_TO_SOT_SMD:SOT-23, F.Cu at (165.5, 135.0)
- added Q9: AO3400A, Package_TO_SOT_SMD:SOT-23, F.Cu at (137.0, 135.0)
- added R1: 10K, Resistor_SMD:R_0805_2012Metric_Pad1.20x1.40mm_HandSolder, F.Cu at (79.4, 112.0)
- added R10: 100k, Resistor_SMD:R_0603_1608Metric_Pad0.98x0.95mm_HandSolder, F.Cu at (187.3, 109.4)
- added R11: 22k, Resistor_SMD:R_0603_1608Metric_Pad0.98x0.95mm_HandSolder, F.Cu at (187.3, 112.3)
- added R12: 100k, Resistor_SMD:R_0603_1608Metric_Pad0.98x0.95mm_HandSolder, F.Cu at (209.5, 125.5)
- added R13: 13.3k, Resistor_SMD:R_0603_1608Metric_Pad0.98x0.95mm_HandSolder, F.Cu at (209.5, 128.5)
- added R14: 22, Resistor_SMD:R_0805_2012Metric_Pad1.20x1.40mm_HandSolder, F.Cu at (91.2, 84.5)
- added R15: 22, Resistor_SMD:R_0805_2012Metric_Pad1.20x1.40mm_HandSolder, F.Cu at (91.2, 87.5)
- added R16: 10k, Resistor_SMD:R_0805_2012Metric_Pad1.20x1.40mm_HandSolder, F.Cu at (91.2, 90.4)
- added R17: 10k, Resistor_SMD:R_0805_2012Metric_Pad1.20x1.40mm_HandSolder, F.Cu at (79.4, 117.9)
- added R18: 10K, Resistor_SMD:R_0805_2012Metric_Pad1.20x1.40mm_HandSolder, F.Cu at (79.4, 120.8)
- added R19: 10K, Resistor_SMD:R_0805_2012Metric_Pad1.20x1.40mm_HandSolder, F.Cu at (79.4, 123.8)
- added R2: 10K, Resistor_SMD:R_0805_2012Metric_Pad1.20x1.40mm_HandSolder, F.Cu at (79.4, 114.9)
- added R20: 10K, Resistor_SMD:R_0805_2012Metric_Pad1.20x1.40mm_HandSolder, F.Cu at (79.4, 126.7)
- added R21: 10K, Resistor_SMD:R_0805_2012Metric_Pad1.20x1.40mm_HandSolder, F.Cu at (79.4, 129.7)
- added R22: 10K, Resistor_SMD:R_0805_2012Metric_Pad1.20x1.40mm_HandSolder, F.Cu at (182.1, 136.7)
- added R23: 100k, Resistor_SMD:R_0805_2012Metric_Pad1.20x1.40mm_HandSolder, F.Cu at (153.0, 135.0)
- added R24: 100, Resistor_SMD:R_0805_2012Metric_Pad1.20x1.40mm_HandSolder, F.Cu at (151.0, 135.0)
- added R25: 100, Resistor_SMD:R_0805_2012Metric_Pad1.20x1.40mm_HandSolder, F.Cu at (141.5, 135.0)
- added R26: 100k, Resistor_SMD:R_0805_2012Metric_Pad1.20x1.40mm_HandSolder, F.Cu at (143.5, 135.0)
- added R27: 100, Resistor_SMD:R_0805_2012Metric_Pad1.20x1.40mm_HandSolder, F.Cu at (160.5, 135.0)
- added R28: 100k, Resistor_SMD:R_0805_2012Metric_Pad1.20x1.40mm_HandSolder, F.Cu at (162.5, 135.0)
- added R29: 100, Resistor_SMD:R_0805_2012Metric_Pad1.20x1.40mm_HandSolder, F.Cu at (132.0, 135.0)
- added R30: 100k, Resistor_SMD:R_0805_2012Metric_Pad1.20x1.40mm_HandSolder, F.Cu at (134.0, 135.0)
- added R5: 1K, Resistor_SMD:R_0805_2012Metric_Pad1.20x1.40mm_HandSolder, F.Cu at (189.5, 55.5)
- added R6: 49.9K, Resistor_SMD:R_0805_2012Metric_Pad1.20x1.40mm_HandSolder, F.Cu at (182.1, 130.7)
- added R7: 5.1K, Resistor_SMD:R_0805_2012Metric_Pad1.20x1.40mm_HandSolder, F.Cu at (179.6, 130.7)
- added U2: HUSB238_xxxDD, Package_DFN_QFN:WDFN-10-1EP_3x3mm_P0.5mm_EP1.8x2.5mm_ThermalVias, F.Cu at (177.5, 135.0)
- added U3: TPS54302, Package_TO_SOT_SMD:SOT-23-6, F.Cu at (187.3, 100.8)
- added U4: TPS54302, Package_TO_SOT_SMD:SOT-23-6, F.Cu at (209.5, 116.9)
- C5: value 1u -> 100n
- C6: value 1n -> 100n
- D3: footprint Diode_SMD:D_SOD-123F -> fertilizer-pump:D_SOD-123FL
- J1: value Conn_01x04 -> Stepper1
- J2: value Conn_01x04 -> Stepper2
- R8: value 10k -> 10.5K
- moved A1 110.8 mm to (218.8, 101.9), turned to 180 degrees
- moved A2 88.9 mm to (218.3, 74.9), turned to 180 degrees
- moved J2 60.2 mm to (225.0, 62.2), turned to -90 degrees
- moved C5 38.2 mm to (172.6, 99.9)
- moved C6 38.2 mm to (172.6, 102.9)
- moved U1 37.9 mm to (177.1, 61.6)
- moved R8 36.3 mm to (182.1, 134.7), turned to 180 degrees
- moved J1 34.0 mm to (225.5, 89.2), turned to -90 degrees
- moved J6 33.0 mm to (177.5, 148.5)
- moved D1 30.1 mm to (177.5, 141.0), turned to 90 degrees
- moved D2 29.2 mm to (171.0, 141.5), turned to 180 degrees
- moved D3 27.1 mm to (187.0, 148.5), turned to -90 degrees
- renumbered U2 to U1
Connections:
- net +12V renamed VMotor
- A1 pad 1: DRIV.ENABLE -> ~{DRIV1.ENABLE}
- A2 pad 1: DRIV.ENABLE -> ~{DRIV2.ENABLE}
- C5 pad 1: USB.VBUS -> Net-(U3-SW)
- C5 pad 2: GND -> Net-(U3-BOOT)
- C6 pad 1: Net-(J6-SHIELD) -> VRegulator
- R8 pad 1: +3.3V -> GND
- R8 pad 2: I^{2}C.SCL -> Net-(U2-ISET)
- U1 pad 10: unconnected-(U2-GPIO17/U1TXD/ADC2_CH6-Pad10) -> DRIV4.DIR
- U1 pad 11: unconnected-(U2-GPIO18/U1RXD/ADC2_CH7/CLK_OUT3-Pad11) -> I^{2}C.SDA
- U1 pad 13: unconnected-(U2-GPIO19/U1RTS/ADC2_CH8/CLK_OUT2/USB_D--Pad13) -> Net-(U1-GPIO19/U1RTS/ADC2_CH8/CLK_OUT2/USB_D-)
- U1 pad 14: unconnected-(U2-GPIO20/U1CTS/ADC2_CH9/CLK_OUT1/USB_D+-Pad14) -> Net-(U1-GPIO20/U1CTS/ADC2_CH9/CLK_OUT1/USB_D+)
- U1 pad 18: unconnected-(U2-GPIO10/TOUCH10/ADC1_CH9/FSPICS0/FSPIIO4/SUBSPICS0-Pad18) -> ~{DRIV3.ENABLE}
- U1 pad 19: unconnected-(U2-GPIO11/TOUCH11/ADC2_CH0/FSPID/FSPIIO5/SUBSPID-Pad19) -> DRIV3.STEP
- U1 pad 2: unconnected-(U2-3V3-Pad2) -> +3.3V
- U1 pad 20: unconnected-(U2-GPIO12/TOUCH12/ADC2_CH1/FSPICLK/FSPIIO6/SUBSPICLK-Pad20) -> DRIV3.DIR
- U1 pad 21: unconnected-(U2-GPIO13/TOUCH13/ADC2_CH2/FSPIQ/FSPIIO7/SUBSPIQ-Pad21) -> ~{DRIV4.ENABLE}
- U1 pad 22: unconnected-(U2-GPIO14/TOUCH14/ADC2_CH3/FSPIWP/FSPIDQS/SUBSPIWP-Pad22) -> DRIV4.STEP
- U1 pad 23: unconnected-(U2-GPIO21-Pad23) -> I^{2}C.SCL
- U1 pad 24: unconnected-(U2-GPIO47/SPICLK_P/SUBSPICLK_P_DIFF-Pad24) -> SERVO4.PWM
- U1 pad 27: unconnected-(U2-GPIO0/BOOT-Pad27) -> ESP_BOOT
- U1 pad 3: unconnected-(U2-EN-Pad3) -> ESP_EN
- U1 pad 31: unconnected-(U2-GPIO38/FSPIWP/SUBSPIWP-Pad31) -> SERVO1.PWM
- U1 pad 32: unconnected-(U2-MTCK/GPIO39/CLK_OUT3/SUBSPICS1-Pad32) -> SERVO2.PWM
- U1 pad 33: unconnected-(U2-MTDO/GPIO40/CLK_OUT2-Pad33) -> SERVO3.PWM
- U1 pad 38: DRIV.UART.RX_{uC} -> DRIV.UART
Other:
- board size 150 x 100 mm -> 100 x 100 mm

Commit message: arrange components
Parts:
- added H1: MountingHole, MountingHole:MountingHole_3.2mm_M3_Pad_Via, F.Cu at (134.2, 54.2)
- added H2: MountingHole, MountingHole:MountingHole_3.2mm_M3_Pad_Via, F.Cu at (225.8, 54.2)
- added H3: MountingHole, MountingHole:MountingHole_3.2mm_M3_Pad_Via, F.Cu at (225.8, 145.8)
- added H4: MountingHole, MountingHole:MountingHole_3.2mm_M3_Pad_Via, F.Cu at (134.2, 145.8)
- moved C10 119.8 mm to (64.0, 165.5)
- moved C11 119.8 mm to (69.6, 153.8)
- moved C5 119.8 mm to (64.0, 150.5)
- moved C6 119.8 mm to (64.0, 153.5)
- moved C7 119.8 mm to (64.0, 156.5)
- moved C8 119.8 mm to (64.0, 159.5)
- moved C9 119.8 mm to (64.0, 162.5)
- moved L1 119.8 mm to (71.4, 162.6)
- moved U3 119.8 mm to (78.7, 151.4)
- moved R10 119.8 mm to (78.7, 160.0)
- moved R11 119.8 mm to (78.7, 163.0)
- moved J4 107.1 mm to (225.0, 125.2), turned to -90 degrees
- moved C16 95.7 mm to (104.9, 160.8)
- moved C12 95.7 mm to (104.9, 148.7)
- moved C13 95.7 mm to (104.9, 151.7)
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Connections:
- D1 pad 1: USB.D+ -> USB.D-
- D1 pad 2: USB.D- -> USB.D+
- D2 pad 1: USB.CC1 -> USB.CC2
- D2 pad 2: USB.CC2 -> USB.CC1
Routing:
- net USB.VBUS: track 0.00 -> 35.4 mm
- net BJ_Power: track 0.00 -> 29.6 mm
- net USB.CC2: track 0.00 -> 23.0 mm
- net USB.CC1: track 0.00 -> 13.0 mm, vias 0 -> 2
- net Net-(Q1-G): track 0.00 -> 6.20 mm
- net USB.D+: track 0.00 -> 5.34 mm
- net USB.D-: track 0.00 -> 5.34 mm
- net Net-(JP1-B): track 0.00 -> 5.34 mm
- net Net-(JP2-B): track 0.00 -> 3.85 mm
- net Net-(U2-VSET): track 0.00 -> 2.85 mm
- net Net-(U2-GATE): track 0.00 -> 2.53 mm
- net Net-(U2-ISET): track 0.00 -> 1.91 mm
- net GND: vias 0 -> 5
- added copper zone on B.Cu, net GND
- added copper zone on F.Cu, net GND
Other:
- outline, holes or cut-outs redrawn
