File: KiCad/power.kicad_sch (KiCad schematic)
At the start: 15 parts, among them J6 USB_C_Receptacle_USB2.0_16P, Q1 PMOS, U1 HUSB238_xxxDD

Commit message: add buck converter, fix footprints
Parts:
- added C10, C16, C17, C9: 22u, Capacitor_SMD:C_0805_2012Metric_Pad1.18x1.45mm_HandSolder, symbol Device:C_Small
- added C11, C18: 220uF, Capacitor_THT:CP_Radial_D8.0mm_P3.50mm, symbol Device:C_Polarized_Small
- added C12, C13, C5, C6: 100n, Capacitor_SMD:C_0805_2012Metric_Pad1.18x1.45mm_HandSolder, symbol Device:C_Small
- added C14, C7: 10u, Capacitor_SMD:C_0805_2012Metric_Pad1.18x1.45mm_HandSolder, symbol Device:C_Small
- added C15: 75p, Capacitor_SMD:C_0805_2012Metric_Pad1.18x1.45mm_HandSolder, symbol Device:C_Small
- added C8: 47p, Capacitor_SMD:C_0805_2012Metric_Pad1.18x1.45mm_HandSolder, symbol Device:C_Small
- added L1, L2: 10u, Inductor_SMD:L_APV_APH0630, symbol Device:L
- added R10, R12: 100k, Resistor_SMD:R_0805_2012Metric_Pad1.20x1.40mm_HandSolder, symbol Device:R_Small
- added R11: 22k, Resistor_SMD:R_0805_2012Metric_Pad1.20x1.40mm_HandSolder, symbol Device:R_Small
- added R13: 13.3k, Resistor_SMD:R_0805_2012Metric_Pad1.20x1.40mm_HandSolder, symbol Device:R_Small
- added U3, U4: TPS54302, Package_TO_SOT_SMD:SOT-23-6, symbol Regulator_Switching:TPS54202DDC
- D3: footprint Diode_SMD:D_SOD-123F -> fertilizer-pump:D_SOD-123FL
- renumbered C5 to C3, C6 to C4, JP2 to JP1, JP1 to JP2, R5 to R8, R4 to R9, U1 to U2
Connections:
- net GND: now also C10.2, C11.2, C13.2, C14.2, C16.2, C17.2, C18.2, C6.2, C7.2, C9.2, R11.2, R13.2, U3.1 (GND), U4.1 (GND)
- net PD_Power: now also C13.1, C14.1, C6.1, C7.1, U3.3 (VIN), U4.3 (VIN)
- net I2C.SCL renamed I^{2}C.SCL
- net I2C.SDA renamed I^{2}C.SDA
- new net: C8.2, R10.2, R11.1, U3.4 (FB)
- new net: C5.1, L1.1, U3.2 (SW)
- new net: C5.2, U3.6 (BOOT)
- new net: C12.1, L2.1, U4.2 (SW)
- new net: C12.2, U4.6 (BOOT)
- new net: C15.2, R12.2, R13.1, U4.4 (FB)
- new net +3.3V: C10.1, C11.1, C8.1, C9.1, L1.2, R10.1
- new net +5V: C15.1, C16.1, C17.1, C18.1, L2.2, R12.1
- no-connect marks 2 -> 4
Other:
- note added: "(100k*0.596V)/(3.3V-0.596V)= 22K"
- note added: "(100k*0.596V)/(5V-0.596V)= 13.53K"
- note added: "R20 = @{round(${/156e031f-7691-48a3-975c-ba45ae33e444/86a463a5-ffcd-42ab-ac8e-5a7cf12baa21/ef7e9748-2f48-4060-acbc-2f18b3e1a9ab:VALUE} * 0.596 / (5 - 0.596) / 1000,3)}kΩ"
- note added: "R22 = @{round(${/156e031f-7691-48a3-975c-ba45ae33e444/86a463a5-ffcd-42ab-ac8e-5a7cf12baa21/1e88ea33-3cb9-422e-8a77-5b57b038368d:VALUE} * 0.596 / (3.3 - 0.596) / 1000, 3)}kΩ"
- note removed: "FIX: wrong footprint SOD123FL instead of SOD123F"

Commit message: add valve driver, many changes
Parts:
- removed Q1: PMOS, symbol Simulation_SPICE:PMOS
- removed R9: 10K, symbol Device:R_Small
- added J15: Barrel_Jack_Switch, Connector_BarrelJack:BarrelJack_GCT_DCJ200-10-A_Horizontal, symbol Connector:Barrel_Jack_Switch
- added JP8: VMotor source select, Jumper:SolderJumper-3_P1.3mm_Open_RoundedPad1.0x1.5mm, symbol Jumper:SolderJumper_3_Open
- added JP9: VRegulator source select, Jumper:SolderJumper-3_P1.3mm_Open_RoundedPad1.0x1.5mm, symbol Jumper:SolderJumper_3_Open
- added Q1: SI2307A, Package_TO_SOT_SMD:SOT-23, symbol Transistor_FET:Q_PMOS_GSD
- added R22: 10K, Resistor_SMD:R_0805_2012Metric_Pad1.20x1.40mm_HandSolder, symbol Device:R_Small
- C11, C18, C4: now not fitted
- C3: LCSC (none) -> C89190
- JP1, JP2, JP3: footprint (none) -> Jumper:SolderJumper-2_P1.3mm_Open_RoundedPad1.0x1.5mm
- R10, R12: footprint Resistor_SMD:R_0805_2012Metric_Pad1.20x1.40mm_HandSolder -> Resistor_SMD:R_0603_1608Metric_Pad0.98x0.95mm_HandSolder; LCSC C3017875 -> C51048119
- R11: footprint Resistor_SMD:R_0805_2012Metric_Pad1.20x1.40mm_HandSolder -> Resistor_SMD:R_0603_1608Metric_Pad0.98x0.95mm_HandSolder; LCSC C2907309 -> C54102214
- R13: footprint Resistor_SMD:R_0805_2012Metric_Pad1.20x1.40mm_HandSolder -> Resistor_SMD:R_0603_1608Metric_Pad0.98x0.95mm_HandSolder; LCSC C3017875 -> C858840
- R6: footprint (none) -> Resistor_SMD:R_0805_2012Metric_Pad1.20x1.40mm_HandSolder; LCSC (none) -> C2930203
- R7: footprint (none) -> Resistor_SMD:R_0805_2012Metric_Pad1.20x1.40mm_HandSolder; LCSC (none) -> C118848
- R8: footprint (none) -> Resistor_SMD:R_0805_2012Metric_Pad1.20x1.40mm_HandSolder; LCSC (none) -> C40086
Connections:
- net GND: now also J15.2, J15.3, R22.1
- net PD_Power: now also JP8.3 (B), JP9.3 (B), Q1.3 (D); no longer C13.1, C14.1, C6.1, C7.1, U3.3 (VIN), U4.3 (VIN)
- net USB.VBUS: now also Q1.2 (S)
- net at R6.1, R7.2: now also Q1.1 (G)
- net at U2.8 (VSET): now also R22.2
- new net BJ_Power: J15.1, JP8.1 (A), JP9.1 (A)
- new net VMotor: JP8.2 (C)
- new net VRegulator: C13.1, C14.1, C6.1, C7.1, JP9.2 (C), U3.3 (VIN), U4.3 (VIN)
Other:
- note added: "If Powerdelivery not working"

Commit message: arrange components
Parts:
- added H1, H2, H3, H4: MountingHole, MountingHole:MountingHole_3.2mm_M3_Pad_Via, symbol Mechanical:MountingHole
Connections:
- net USB.CC1: now also D2.2 (A2); no longer D2.1 (A1)
- net USB.CC2: now also D2.1 (A1); no longer D2.2 (A2)
- net USB.D+: now also D1.2 (A2); no longer D1.1 (A1)
- net USB.D-: now also D1.1 (A1); no longer D1.2 (A2)
