File: KiCad/stepper.kicad_sch (KiCad schematic)
At the start: 12 parts, among them J1 Stepper1, J2 Stepper2, J3 Servo, J4 Stepper2, J5 Stepper2

Commit message: add buck converter, fix footprints
Parts:
- added J7: Servo2, symbol Connector_Generic:Conn_01x03
- added J8: Servo3, symbol Connector_Generic:Conn_01x03
- added J9: Servo4, symbol Connector_Generic:Conn_01x03
- J5: renamed from J3; value Servo -> Servo1
- renumbered C7 to C2, J4 to J3, J5 to J4, R1 to R5
Connections:
- net +3.3V: now also A3.3 (MS2), A4.3 (MS2); no longer A3.2 (MS1)
- net +5V: now also J7.1 (Pin_1), J8.1 (Pin_1), J9.1 (Pin_1)
- net DRIV2.A1: no longer A4.13 (A1), J3.4 (Pin_4), J4.4 (Pin_4)
- net DRIV2.A2: no longer A4.14 (A2), J3.2 (Pin_2), J4.2 (Pin_2)
- net DRIV2.B1: no longer A4.12 (B1), J3.3 (Pin_3), J4.3 (Pin_3)
- net DRIV2.B2: no longer A4.11 (B2), J3.1 (Pin_1), J4.1 (Pin_1)
- net DRIV2.DIAG: no longer A3.17 (DIAG), A4.17 (DIAG)
- net DRIV2.DIR: no longer A3.8 (DIR), A4.8 (DIR)
- net DRIV2.STEP: no longer A3.7 (STEP), A4.7 (STEP)
- net DRIV3.A1: now also J3.4 (Pin_4)
- net DRIV3.A2: now also J3.2 (Pin_2)
- net DRIV3.B1: now also J3.3 (Pin_3)
- net DRIV3.B2: now also J3.1 (Pin_1)
- net GND: now also A3.2 (MS1), J7.3 (Pin_3), J8.3 (Pin_3), J9.3 (Pin_3); no longer A3.3 (MS2), A4.3 (MS2)
- net +12V renamed PD_Power
- removed net DRIV.ENABLE: A1.1 (ENABLE), A2.1 (ENABLE), A3.1 (ENABLE), A4.1 (ENABLE)
- new net DRIV3.DIAG: A3.17 (DIAG)
- new net DRIV3.DIR: A3.8 (DIR)
- new net DRIV3.STEP: A3.7 (STEP)
- new net DRIV4.A1: A4.13 (A1), J4.4 (Pin_4)
- new net DRIV4.A2: A4.14 (A2), J4.2 (Pin_2)
- new net DRIV4.B1: A4.12 (B1), J4.3 (Pin_3)
- new net DRIV4.B2: A4.11 (B2), J4.1 (Pin_1)
- new net DRIV4.DIAG: A4.17 (DIAG)
- new net DRIV4.DIR: A4.8 (DIR)
- new net DRIV4.STEP: A4.7 (STEP)
- new net SERVO2.PWM: J7.2 (Pin_2)
- new net SERVO3.PWM: J8.2 (Pin_2)
- new net SERVO4.PWM: J9.2 (Pin_2)
- new net ~{DRIV1.ENABLE}: A1.1 (ENABLE)
- new net ~{DRIV2.ENABLE}: A2.1 (ENABLE)
- new net ~{DRIV3.ENABLE}: A3.1 (ENABLE)
- new net ~{DRIV4.ENABLE}: A4.1 (ENABLE)
Other:
- moved on the sheet: J5

Commit message: add valve driver, many changes
Parts:
- added C23, C25, C27: 220µF, Capacitor_SMD:CP_Elec_6.3x7.7, symbol Device:C_Polarized
- added C24, C26, C28: 100n, Capacitor_SMD:C_0805_2012Metric_Pad1.18x1.45mm_HandSolder, symbol Device:C_Small
- added J11, J12, J13, J14: Conn_01x02, Connector_JST:JST_XH_B2B-XH-A_1x02_P2.50mm_Vertical, symbol Connector_Generic:Conn_01x02
- C1: value 100u -> 220µF; footprint (none) -> Capacitor_SMD:CP_Elec_6.3x7.7; LCSC (none) -> C7471881
- C2: LCSC (none) -> C48579601
- J3: value Stepper2 -> Stepper3
- J4: value Stepper2 -> Stepper4
- J5, J7, J8, J9: footprint (none) -> Connector_JST:JST_XH_B3B-XH-A_1x03_P2.50mm_Vertical
- R5: footprint (none) -> Resistor_SMD:R_0805_2012Metric_Pad1.20x1.40mm_HandSolder; LCSC (none) -> C54921120
Connections:
- net GND: now also C23.2, C24.2, C25.2, C26.2, C27.2, C28.2
- net PD_Power: now also J11.1 (Pin_1), J12.1 (Pin_1), J13.1 (Pin_1), J14.1 (Pin_1); no longer A1.16 (VM), A2.16 (VM), A3.16 (VM), A4.16 (VM), C1.1, C2.1
- net DRIV.UART.TX renamed DRIV.UART.TX_{MCU}
- new net VALVE1.OUT: J11.2 (Pin_2)
- new net VALVE2.OUT: J12.2 (Pin_2)
- new net VALVE3.OUT: J13.2 (Pin_2)
- new net VALVE4.OUT: J14.2 (Pin_2)
- new net VMotor: A1.16 (VM), A2.16 (VM), A3.16 (VM), A4.16 (VM), C1.1, C2.1, C23.1, C24.1, C25.1, C26.1, C27.1, C28.1
Other:
- added sheet valve_drive_channel (valve_drive_channel.kicad_sch)
- added sheet valve_drive_channel1 (valve_drive_channel.kicad_sch)
- added sheet valve_drive_channel2 (valve_drive_channel.kicad_sch)
- added sheet valve_drive_channel3 (valve_drive_channel.kicad_sch)
- note added: "Servo"
- moved on the sheet: A2, A3, A4, C2, J2, J3, J4

Commit message: arrange components
Connections:
- net PD_Power is gone; now on net VMotor: J11.1 (Pin_1), J12.1 (Pin_1), J13.1 (Pin_1), J14.1 (Pin_1)
- net DRIV1.A1: now also J1.1 (Pin_1); no longer J1.4 (Pin_4)
- net DRIV1.B1: now also J1.4 (Pin_4); no longer J1.3 (Pin_3)
- net DRIV1.B2: now also J1.3 (Pin_3); no longer J1.1 (Pin_1)
- net DRIV2.A1: now also J2.1 (Pin_1); no longer J2.4 (Pin_4)
- net DRIV2.B1: now also J2.4 (Pin_4); no longer J2.3 (Pin_3)
- net DRIV2.B2: now also J2.3 (Pin_3); no longer J2.1 (Pin_1)
- net DRIV3.A1: now also J3.1 (Pin_1); no longer J3.4 (Pin_4)
- net DRIV3.B1: now also J3.4 (Pin_4); no longer J3.3 (Pin_3)
- net DRIV3.B2: now also J3.3 (Pin_3); no longer J3.1 (Pin_1)
- net DRIV4.A1: now also J4.1 (Pin_1); no longer J4.4 (Pin_4)
- net DRIV4.B1: now also J4.4 (Pin_4); no longer J4.3 (Pin_3)
- net DRIV4.B2: now also J4.3 (Pin_3); no longer J4.1 (Pin_1)
